Commit message: 完善双IMU与双电机分层控制，修复数据质量和时效审核问题

File: ros2_ws/src/mech_bringup/config/dm4340_velocity.urdf.xacro (robot description, xacro)
@@ -11,4 +11,9 @@
   <xacro:arg name="velocity_feedforward_nm" default="0"/>
   <xacro:arg name="velocity_kd" default="3"/>
+  <xacro:arg name="position_kp" default="1"/>
+  <xacro:arg name="position_kd" default="0.2"/>
+  <xacro:arg name="max_target_error_rad" default="0.3"/>
+  <xacro:property name="dm_position_kp" value="$(arg position_kp)"/>
+  <xacro:property name="dm_position_kd" value="$(arg position_kd)"/>
   <xacro:arg name="command_mode" default="velocity"/>
   <xacro:arg name="supervised_effort_bench" default="false"/>
@@ -64,9 +69,10 @@
       <param name="position_min_rad">-12.5</param>
       <param name="position_max_rad">12.5</param>
-      <param name="max_target_error_rad">0.3</param>
-      <param name="kp">0</param>
-      <param name="kd">${0 if dm_command_mode == 'effort' else dm_velocity_kd}</param>
+      <param name="position_guard_margin_rad">0.02</param>
+      <param name="max_target_error_rad">$(arg max_target_error_rad)</param>
+      <param name="kp">${dm_position_kp if dm_command_mode == 'position' else 0}</param>
+      <param name="kd">${0 if dm_command_mode == 'effort' else (dm_position_kd if dm_command_mode == 'position' else dm_velocity_kd)}</param>
       <param name="velocity_feedforward_nm">$(arg velocity_feedforward_nm)</param>
-      <param name="max_command_velocity_rad_s">${0 if dm_command_mode == 'effort' else 1.5}</param>
+      <param name="max_command_velocity_rad_s">${0 if dm_command_mode != 'velocity' else 1.5}</param>
       <param name="max_feedback_velocity_rad_s">2</param>
       <param name="max_feedback_torque_nm">5</param>
@@ -80,7 +86,10 @@
         <command_interface name="effort"/>
       </xacro:if>
-      <xacro:unless value="${dm_command_mode == 'effort'}">
+      <xacro:if value="${dm_command_mode == 'velocity'}">
         <command_interface name="velocity"/>
-      </xacro:unless>
+      </xacro:if>
+      <xacro:if value="${dm_command_mode == 'position'}">
+        <command_interface name="position"/>
+      </xacro:if>
       <command_interface name="command_generation"/>
       <state_interface name="position"/>
